File: Hardware/LoRa_irrigation_system/LoRa_irrigation_system.kicad_pcb (KiCad board)
At the start: 2 copper layers, 93.5 x 77.5 mm, 14 parts, among them J1 12VIN, J2 SoilMoisture sensor, J3 WaterPump connector, J4 Conn_Coaxial, K2 SANYOU_SRD_Form_C, U1 LM2596_buck_converter, U2 RASPBERRY_PI_PICO, U4 RFM69HCW LoRa module

Commit message: SWare start
Connections:
- U2 pad GP0: unconnected-(U2-PadGP0) -> RESET
- U2 pad GP1: unconnected-(U2-PadGP1) -> NSS
- U2 pad GP5: NSS -> DIO0
- U4 pad 14: unconnected-(U4-DIO0-Pad14) -> DIO0
Routing:
- net DIO0: track 0.00 -> 61.3 mm
- net RESET: track 0.00 -> 15.4 mm
- net NSS: track 0.00 -> 15.1 mm
Changed lines of the file:
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@@
 	(net 16 "SCK")
 	(net 17 "MOSI")
-	(net 18 "unconnected-(U2-PadGP1)")
+	(net 18 "DIO0")
 	(net 19 "NSS")
 	(net 20 "MISO")
@@
 	(net 26 "unconnected-(U2-Pad3V3_EN)")
 	(net 27 "unconnected-(U2-PadGP27_A1)")
-	(net 28 "unconnected-(U2-PadGP0)")
-	(net 29 "unconnected-(U2-PadGP17)")
-	(net 30 "unconnected-(U2-PadGP7)")
-	(net 31 "unconnected-(U2-Pad3V3)")
-	(net 32 "unconnected-(U2-PadRUN)")
-	(net 33 "unconnected-(U2-PadADC_VREF)")
-	(net 34 "unconnected-(U4-DIO5-Pad7)")
-	(net 35 "unconnected-(U4-DIO4-Pad12)")
-	(net 36 "unconnected-(U4-DIO0-Pad14)")
-	(net 37 "unconnected-(U4-DIO3-Pad11)")
-	(net 38 "unconnected-(U4-DIO1-Pad15)")
-	(net 39 "RESET")
-	(net 40 "unconnected-(U4-DIO2-Pad16)")
-	(net 41 "unconnected-(K2-Pad4)")
-	(net 42 "IrrigON")
-	(net 43 "unconnected-(U2-PadGP21)")
-	(net 44 "unconnected-(U2-PadGP13)")
-	(net 45 "unconnected-(U2-PadGP12)")
-	(net 46 "unconnected-(U2-PadGP11)")
-	(net 47 "unconnected-(U2-PadGP16)")
+	(net 28 "unconnected-(U2-PadGP17)")
+	(net 29 "unconnected-(U2-PadGP7)")
+	(net 30 "unconnected-(U2-Pad3V3)")
+	(net 31 "unconnected-(U2-PadRUN)")
+	(net 32 "unconnected-(U2-PadADC_VREF)")
+	(net 33 "unconnected-(U4-DIO5-Pad7)")
+	(net 34 "unconnected-(U4-DIO4-Pad12)")
+	(net 35 "unconnected-(U4-DIO3-Pad11)")
+	(net 36 "unconnected-(U4-DIO1-Pad15)")
+	(net 37 "RESET")
+	(net 38 "unconnected-(U4-DIO2-Pad16)")
+	(net 39 "unconnected-(K2-Pad4)")
+	(net 40 "IrrigON")
+	(net 41 "unconnected-(U2-PadGP21)")
+	(net 42 "unconnected-(U2-PadGP13)")
+	(net 43 "unconnected-(U2-PadGP12)")
+	(net 44 "unconnected-(U2-PadGP11)")
+	(net 45 "unconnected-(U2-PadGP16)")
 	(footprint "Connector_Coaxial:SMA_Amphenol_132134_Vertical"
 		(layer "F.Cu")
@@
 			(layers "*.Cu" "*.Mask")
 			(remove_unused_layers no)
-			(net 31 "unconnected-(U2-Pad3V3)")
+			(net 30 "unconnected-(U2-Pad3V3)")
 			(pinfunction "3V3")
 			(pintype "bidirectional")
@@
 			(layers "*.Cu" "*.Mask")
 			(remove_unused_layers no)
-			(net 33 "unconnected-(U2-PadADC_VREF)")
+			(net 32 "unconnected-(U2-PadADC_VREF)")
 			(pinfunction "ADC_VREF")
 			(pintype "bidirectional")
@@
 			(layers "*.Cu" "*.Mask")
 			(remove_unused_layers no)
-			(net 28 "unconnected-(U2-PadGP0)")
+			(net 37 "RESET")
 			(pinfunction "GP0")
 			(pintype "bidirectional")
@@
 			(layers "*.Cu" "*.Mask")
 			(remove_unused_layers no)
-			(net 18 "unconnected-(U2-PadGP1)")
+			(net 19 "NSS")
 			(pinfunction "GP1")
 			(pintype "bidirectional")
@@
 			(layers "*.Cu" "*.Mask")
 			(remove_unused_layers no)
-			(net 19 "NSS")
+			(net 18 "DIO0")
 			(pinfunction "GP5")
 			(pintype "bidirectional")
@@
 			(layers "*.Cu" "*.Mask")
 			(remove_unused_layers no)
-			(net 30 "unconnected-(U2-PadGP7)")
+			(net 29 "unconnected-(U2-PadGP7)")
 			(pinfunction "GP7")
 			(pintype "bidirectional")
@@
 			(layers "*.Cu" "*.Mask")
 			(remove_unused_layers no)
-			(net 46 "unconnected-(U2-PadGP11)")
+			(net 44 "unconnected-(U2-PadGP11)")
 			(pinfunction "GP11")
 			(pintype "bidirectional")
@@
 			(layers "*.Cu" "*.Mask")
 			(remove_unused_layers no)
-			(net 45 "unconnected-(U2-PadGP12)")
+			(net 43 "unconnected-(U2-PadGP12)")
 			(pinfunction "GP12")
 			(pintype "bidirectional")
@@
 			(layers "*.Cu" "*.Mask")
 			(remove_unused_layers no)
-			(net 44 "unconnected-(U2-PadGP13)")
+			(net 42 "unconnected-(U2-PadGP13)")
 			(pinfunction "GP13")
 			(pintype "bidirectional")
@@
 			(layers "*.Cu" "*.Mask")
 			(remove_unused_layers no)
-			(net 47 "unconnected-(U2-PadGP16)")
+			(net 45 "unconnected-(U2-PadGP16)")
 			(pinfunction "GP16")
 			(pintype "bidirectional")
@@
 			(layers "*.Cu" "*.Mask")
 			(remove_unused_layers no)
-			(net 29 "unconnected-(U2-PadGP17)")
+			(net 28 "unconnected-(U2-PadGP17)")
 			(pinfunction "GP17")
 			(pintype "bidirectional")
@@
 			(layers "*.Cu" "*.Mask")
 			(remove_unused_layers no)
-			(net 42 "IrrigON")
+			(net 40 "IrrigON")
 			(pinfunction "GP20")
 			(pintype "bidirectional")
@@
 			(layers "*.Cu" "*.Mask")
 			(remove_unused_layers no)
-			(net 43 "unconnected-(U2-PadGP21)")
+			(net 41 "unconnected-(U2-PadGP21)")
 			(pinfunction "GP21")
 			(pintype "bidirectional")
@@
 			(layers "*.Cu" "*.Mask")
 			(remove_unused_layers no)
-			(net 32 "unconnected-(U2-PadRUN)")
+			(net 31 "unconnected-(U2-PadRUN)")
 			(pinfunction "RUN")
 			(pintype "bidirectional")
@@
 			(layers "*.Cu" "*.Mask")
 			(remove_unused_layers no)
-			(net 41 "unconnected-(K2-Pad4)")
+			(net 39 "unconnected-(K2-Pad4)")
 			(pintype "passive")
 		)
@@
 			(size 3 1.2)
 			(layers "F.Cu" "F.Paste" "F.Mask")
-			(net 39 "RESET")
+			(net 37 "RESET")
 			(pinfunction "RESET")
 			(pintype "bidirectional")
@@
 			(size 3 1.2)
 			(layers "F.Cu" "F.Paste" "F.Mask")
-			(net 34 "unconnected-(U4-DIO5-Pad7)")
+			(net 33 "unconnected-(U4-DIO5-Pad7)")
 			(pinfunction "DIO5")
 			(pintype "bidirectional")
@@
 			(size 3 1.2)
 			(layers "F.Cu" "F.Paste" "F.Mask")
-			(net 37 "unconnected-(U4-DIO3-Pad11)")
+			(net 35 "unconnected-(U4-DIO3-Pad11)")
 			(pinfunction "DIO3")
 			(pintype "bidirectional")
@@
 			(size 3 1.2)
 			(layers "F.Cu" "F.Paste" "F.Mask")
-			(net 35 "unconnected-(U4-DIO4-Pad12)")
+			(net 34 "unconnected-(U4-DIO4-Pad12)")
 			(pinfunction "DIO4")
 			(pintype "bidirectional")
@@
 			(size 3 1.2)
 			(layers "F.Cu" "F.Paste" "F.Mask")
-			(net 36 "unconnected-(U4-DIO0-Pad14)")
+			(net 18 "DIO0")
 			(pinfunction "DIO0")
 			(pintype "bidirectional")
@@
 			(size 3 1.2)
 			(layers "F.Cu" "F.Paste" "F.Mask")
-			(net 38 "unconnected-(U4-DIO1-Pad15)")
+			(net 36 "unconnected-(U4-DIO1-Pad15)")
 			(pinfunction "DIO1")
 			(pintype "bidirectional")
@@
 			(size 3 1.2)
 			(layers "F.Cu" "F.Paste" "F.Mask")
-			(net 40 "unconnected-(U4-DIO2-Pad16)")
+			(net 38 "unconnected-(U4-DIO2-Pad16)")
 			(pinfunction "DIO2")
 			(pintype "bidirectional")
@@
 			(layers "*.Cu" "*.Mask")
 			(remove_unused_layers no)
-			(net 42 "IrrigON")
+			(net 40 "IrrigON")
 			(pintype "passive")
 		)
@@
 	)
 	(segment
+		(start 107 66.5)
+		(end 107 70)
+		(width 0.8)
+		(layer "F.Cu")
+		(net 18)
+	)
+	(segment
+		(start 114.5 77.5)
+		(end 123.5 77.5)
+		(width 0.8)
+		(layer "F.Cu")
+		(net 18)
+	)
+	(segment
+		(start 97.5 59)
+		(end 97 59.5)
+		(width 0.8)
+		(layer "F.Cu")
+		(net 18)
+	)
+	(segment
+		(start 97 59.5)
+		(end 97 64.5)
+		(width 0.8)
+		(layer "F.Cu")
+		(net 18)
+	)
+	(segment
+		(start 99 66.5)
+		(end 107 66.5)
+		(width 0.8)
+		(layer "F.Cu")
+		(net 18)
+	)
+	(segment
+		(start 124.62 63.88)
+		(end 129.11 63.88)
+		(width 0.8)
+		(layer "F.Cu")
+		(net 18)
+	)
+	(segment
+		(start 123.5 77.5)
+		(end 123.5 65)
+		(width 0.8)
+		(layer "F.Cu")
+		(net 18)
+	)
+	(segment
+		(start 97 64.5)
+		(end 99 66.5)
+		(width 0.8)
+		(layer "F.Cu")
+		(net 18)
+	)
+	(segment
+		(start 123.5 65)
+		(end 124.62 63.88)
+		(width 0.8)
+		(layer "F.Cu")
+		(net 18)
+	)
+	(segment
+		(start 107 70)
+		(end 114.5 77.5)
+		(width 0.8)
+		(layer "F.Cu")
+		(net 18)
+	)
+	(segment
+		(start 100.55 59)
+		(end 97.5 59)
+		(width 0.8)
+		(layer "F.Cu")
+		(net 18)
+	)
+	(segment
+		(start 115.55 55)
+		(end 117.587258 55)
+		(width 0.8)
+		(layer "F.Cu")
+		(net 19)
+	)
+	(segment
+		(start 117.587258 55)
+		(end 117.987258 54.6)
+		(width 0.8)
+		(layer "F.Cu")
+		(net 19)
+	)
+	(segment
+		(start 124.32 51.18)
+		(end 129.11 51.18)
+		(width 0.8)
+		(layer "F.Cu")
+		(net 19)
+	)
+	(segment
+		(start 117.987258 54.6)
+		(end 120.9 54.6)
+		(width 0.8)
+		(layer "F.Cu")
+		(net 19)
+	)
+	(segment
+		(start 120.9 54.6)
+		(end 124.32 51.18)
+		(width 0.8)
+		(layer "F.Cu")
+		(net 19)
+	)
+	(segment
 		(start 128.77 61)
 		(end 129.11 61.34)
@@
 	)
 	(segment
+		(start 115.55 53)
+		(end 119.5 53)
+		(width 0.8)
+		(layer "F.Cu")
+		(net 37)
+	)
+	(segment
+		(start 123.86 48.64)
+		(end 129.11 48.64)
+		(width 0.8)
+		(layer "F.Cu")
+		(net 37)
+	)
+	(segment
+		(start 119.5 53)
+		(end 123.86 48.64)
+		(width 0.8)
+		(layer "F.Cu")
+		(net 37)
+	)
+	(segment
 		(start 152.85 84.2)
 		(end 154.15 85.5)
 		(width 0.8)
 		(layer "B.Cu")
-		(net 42)
+		(net 40)
 	)
 	(segment
@@
 		(width 0.8)
 		(layer "B.Cu")
-		(net 42)
+		(net 40)
 	)
 	(zone
@@
 		(min_thickness 0.25)
 		(filled_areas_thickness no)
-		(fill
+		(fill yes
 			(thermal_gap 0.5)
 			(thermal_bridge_width 0.5)
